Commit message: Gripper connected to robots and oriented correctly

File: aprs_description/urdf/fanuc/aprs_fanuc_macro.xacro (robot description, xacro)
@@ -8,4 +8,6 @@
     <!-- Include ROS2 Control macro -->
     <xacro:include filename="$(find aprs_description)/urdf/fanuc/aprs_fanuc.ros2_control.xacro"/>
+    <!-- Inclue gripper macro -->
+    <xacro:include filename="$(find aprs_description)/urdf/vacuum_gripper/vacuum_grippper_macro.xacro"/>
     <xacro:property name="initial_positions_file" default="$(find aprs_description)/config/fanuc_initial_positions.yaml"/>
     <!-- Run fanuc macro -->
@@ -18,4 +20,10 @@
       initial_positions="${xacro.load_yaml(initial_positions_file)}">
     </xacro:aprs_fanuc_ros2_control>
+    <!-- Run gripper macro -->
+    <xacro:vacuum_gripper
+      parent="fanuc_gripper_link"
+      prefix="fanuc"
+      >
+    </xacro:vacuum_gripper>
   </xacro:macro>
 </robot>

File: aprs_description/urdf/fanuc/fanuc_lrmate200id_macro.xacro (robot description, xacro)
@@ -185,4 +185,5 @@
          </inertial>
       </link>
+      <link name="fanuc_gripper_link"/>
    <!--   <link name="tool0" /> -->
       <joint name = "base_joint_" type = "fixed">
@@ -233,4 +234,9 @@
          <limit effort="${joint6effort}" lower="${joint6lower}" upper="${joint6upper}" velocity="${joint6velocity}" />
       </joint>
+      <joint name = "fanuc_link_6_to_gripper" type = "fixed">
+         <origin xyz = "0 0 0" rpy = "0 1.57 0"/>
+         <parent link = "link_6"/>
+         <child link = "fanuc_gripper_link"/>
+      </joint>
       <gazebo reference="fanuc_base_link">
          <material>Gazebo/Grey</material>
@@ -261,4 +267,8 @@
          <turnGravityOff>true</turnGravityOff>
       </gazebo>
+      <gazebo reference="fanuc_gripper_link">
+         <material>Gazebo/Yellow</material>
+         <turnGravityOff>true</turnGravityOff>
+      </gazebo>
   </xacro:macro>
 </robot>

File: aprs_description/urdf/motoman/aprs_motoman_macro.xacro (robot description, xacro)
@@ -8,4 +8,6 @@
     <!-- Include ROS2 Control macro -->
     <xacro:include filename="$(find aprs_description)/urdf/motoman/aprs_motoman.ros2_control.xacro"/>
+    <!-- Inclue gripper macro -->
+    <xacro:include filename="$(find aprs_description)/urdf/vacuum_gripper/vacuum_grippper_macro.xacro"/>
     <xacro:property name="initial_positions_file" default="$(find aprs_description)/config/motoman_initial_positions.yaml"/>
     <!-- Run motoman macro -->
@@ -18,4 +20,10 @@
       initial_positions="${xacro.load_yaml(initial_positions_file)}">
     </xacro:aprs_motoman_ros2_control>
+    <!-- Run gripper macro -->
+    <xacro:vacuum_gripper
+      parent="motoman_gripper_link"
+      prefix="motoman"
+      >
+    </xacro:vacuum_gripper>
   </xacro:macro>
 </robot>

File: aprs_description/urdf/motoman/motoman_sia20_macro.xacro (robot description, xacro)
@@ -37,4 +37,5 @@
 			</collision>
 		</link>
+		<link name="motoman_gripper_link"/>
 		<joint name = "motoman_base_joint" type = "fixed">
 			<origin rpy = "0 0 0" xyz = "0 0 0"/>
@@ -200,11 +201,8 @@
 			<xacro:default_joint_misc/>
 		</joint>
-		<!-- link motoman_tool0-->
-		<link name="motoman_tool0"/>
-		<!-- joint link_t-motoman_tool0 -->
-		<joint name="link_t-motoman_tool0" type="fixed">
-			<origin rpy="0 0 -3.1415" xyz="0 0 0"/>
-			<parent link="link_t"/>
-			<child  link="motoman_tool0"/>
+		<joint name = "motoman_link_t_to_gripper" type = "fixed">
+			<origin xyz = "0 0.02 0" rpy = "-1.57 0 0"/>
+			<parent link = "link_t"/>
+			<child link = "motoman_gripper_link"/>
 		</joint>
   </xacro:macro>

File: aprs_description/urdf/ur/aprs_ur_macro.xacro (robot description, xacro)
@@ -8,4 +8,6 @@
     <!-- Include ROS2 Control macro -->
     <xacro:include filename="$(find aprs_description)/urdf/ur/aprs_ur.ros2_control.xacro"/>
+    <!-- Inclue gripper macro -->
+    <xacro:include filename="$(find aprs_description)/urdf/vacuum_gripper/vacuum_grippper_macro.xacro"/>
     <xacro:property name="initial_positions_file" default="$(find aprs_description)/config/ur_initial_positions.yaml"/>
     <!-- Run ur macro -->
@@ -25,4 +27,10 @@
       initial_positions="${xacro.load_yaml(initial_positions_file)}">
     </xacro:aprs_ur_ros2_control>
+    <!-- Run gripper macro -->
+    <xacro:vacuum_gripper
+      parent="tool0"
+      prefix="ur"
+      >
+    </xacro:vacuum_gripper>
   </xacro:macro>
 </robot>
