Commit message: Working

File: aprs_description/urdf/aprs_lab_robots.urdf.xacro (robot description, xacro)
@@ -11,5 +11,5 @@
   </joint>
   <joint name = "fanuc_world_to_base" type = "fixed">
-    <origin rpy = "0 0 0" xyz = "-0.5222875 -0.073025 0.84455"/>
+    <origin rpy = "0 0 0" xyz = "-0.5222875 -0.073025 0.87455"/>
     <parent link = "world"/>
     <child link = "aprs_fanuc_base_link"/>
@@ -21,5 +21,5 @@
   </joint>
   <joint name = "motoman_world_to_base" type = "fixed">
-    <origin rpy = "0 0 3.14159" xyz = "0.4953 -0.08255 0.84455"/>
+    <origin rpy = "0 0 3.14159" xyz = "0.4953 -0.08255 0.87455"/>
     <parent link = "world"/>
     <child link = "aprs_motoman_base_link"/>

Commit message: Revert "Robots spawning in"
This reverts commit 296f111bd0237314a285628f382dd9d13a2de7d1.

File: aprs_description/urdf/aprs_lab_robots.urdf.xacro (robot description, xacro)
@@ -11,5 +11,5 @@
   </joint>
   <joint name = "fanuc_world_to_base" type = "fixed">
-    <origin rpy = "0 0 0" xyz = "-0.5222875 -0.073025 0.87455"/>
+    <origin rpy = "0 0 0" xyz = "-0.5222875 -0.073025 0.84455"/>
     <parent link = "world"/>
     <child link = "aprs_fanuc_base_link"/>
@@ -21,5 +21,5 @@
   </joint>
   <joint name = "motoman_world_to_base" type = "fixed">
-    <origin rpy = "0 0 3.14159" xyz = "0.4953 -0.08255 0.87455"/>
+    <origin rpy = "0 0 3.14159" xyz = "0.4953 -0.08255 0.84455"/>
     <parent link = "world"/>
     <child link = "aprs_motoman_base_link"/>
@@ -29,4 +29,6 @@
   <xacro:include filename="$(find aprs_description)/urdf/franka/aprs_franka_macro.xacro"/>
   <xacro:include filename="$(find aprs_description)/urdf/motoman/aprs_motoman_macro.xacro"/>
+    <!-- ROS2 Control Plugin -->
+  <xacro:arg name="controllers" default="$(find aprs_description)/config/robot_controllers.yaml" />
   <xacro:aprs_ur
     parent="aprs_ur_base_link">
@@ -39,11 +41,10 @@
     parent="aprs_motoman_base_link">
   </xacro:aprs_motoman>
-  <!-- ROS2 Control Plugin -->
-  <xacro:arg name="controllers" default="$(find aprs_description)/config/robot_controllers.yaml" />
   <gazebo>
-    <plugin filename="libgazebo_ros2_control.so" name="aprs_robots_gazebo_ros2_control">
+    <plugin filename="libgz_ros2_control-system.so" name="gz_ros2_control::GazeboSimROS2ControlPlugin">
       <ros>
       </ros>
       <parameters>$(arg controllers)</parameters>
+      <load_params_directly>true</load_params_directly>
     </plugin>
   </gazebo>

File: aprs_description/urdf/fanuc/aprs_fanuc.ros2_control.xacro (robot description, xacro)
@@ -6,5 +6,5 @@
     <ros2_control name="${name}" type="system">
       <hardware>
-        <plugin>gazebo_ros2_control/GazeboSystem</plugin>
+        <plugin>gz_ros2_control/GazeboSimSystem</plugin>
       </hardware>
       <joint name="joint_1">

File: aprs_description/urdf/franka/aprs_franka.ros2_control.xacro (robot description, xacro)
@@ -6,5 +6,5 @@
     <ros2_control name="${name}" type="system">
       <hardware>
-        <plugin>gazebo_ros2_control/GazeboSystem</plugin>
+        <plugin>gz_ros2_control/GazeboSimSystem</plugin>
       </hardware>
       <joint name="fr3_joint1">

File: aprs_description/urdf/franka/aprs_franka_macro.xacro (robot description, xacro)
@@ -2,4 +2,6 @@
 <robot xmlns:xacro="http://wiki.ros.org/xacro">
   <xacro:macro name="aprs_franka">
+    <!-- Inclue franka robot macro -->
+    <!-- <xacro:include filename="$(find franka_description)/robots/common/franka_robot.xacro"/> -->
     <xacro:include filename="$(find aprs_description)/urdf/franka/aprs_franka.ros2_control.xacro"/>
     <xacro:property name="initial_positions_file" default="$(find aprs_description)/config/franka_initial_positions.yaml"/>
@@ -20,5 +22,5 @@
       inertials="${xacro.load_yaml('$(find aprs_description)/urdf/franka/fr3/inertials.yaml')}">
     </xacro:franka_hand>
-    <!-- Run franka macro -->
+    <!-- Run fanuc macro -->
     <xacro:aprs_franka_ros2_control
       name="franka"

File: aprs_description/urdf/franka/franka_arm.xacro (robot description, xacro)
@@ -2,4 +2,10 @@
 <robot xmlns:xacro="http://www.ros.org/wiki/xacro" name="fer">
   <xacro:include filename="$(find aprs_description)/urdf/franka/utils.xacro" />
+  <!-- safety_distance: Minimum safety distance in [m] by which the collision volumes are expanded and which is enforced during robot motions -->
+  <!-- arm_id: Namespace of the robot arm. Serves to differentiate between arms in case of multiple instances. -->
+  <!-- joint_limits: description of the joint limits that comes from a YAML file. Example definition: ${xacro.load_yaml('$(find franka_description)/robots/fr3/joint_limits.yaml')} -->
+  <!-- kinematics: description of the kinematics that comes from a YAML file. Example definition: ${xacro.load_yaml('$(find franka_description)/robots/fr3/kinematics.yaml')} -->
+  <!-- inertials: description of the inertials that comes from a YAML file. Example definition: ${xacro.load_yaml('$(find franka_description)/robots/fr3/inertials.yaml')} -->
+  <!-- dynamics: description of the dynamics that comes from a YAML file. Example definition: ${xacro.load_yaml('$(find franka_description)/robots/fr3/dynamics.yaml')} -->
   <xacro:macro name="franka_arm" params="arm_id description_pkg:='franka_description' connected_to:='base' xyz:='0 0 0' rpy:='0 0 0' gazebo:=false safety_distance:=0 joint_limits inertials kinematics dynamics with_sc:=false" >
     <xacro:unless value="${not connected_to}">

File: aprs_description/urdf/franka/franka_hand.xacro (robot description, xacro)
@@ -1,4 +1,5 @@
 <?xml version="1.0" encoding="utf-8"?>
 <robot xmlns:xacro="http://www.ros.org/wiki/xacro" name="hand">
+  <!-- safety_distance: Minimum safety distance in [m] by which the collision volumes are expanded and which is enforced during robot motions -->
   <xacro:macro name="franka_hand" params="connected_to:='' arm_id rpy:='0 0 0' xyz:='0 0 0' tcp_xyz:='0 0 0.1034' tcp_rpy:='0 0 0' safety_distance:=0 gazebo:=false description_pkg:=franka_description with_sc:=false inertials">
     <xacro:unless value="${connected_to == ''}">

File: aprs_description/urdf/motoman/aprs_motoman.ros2_control.xacro (robot description, xacro)
@@ -6,5 +6,5 @@
     <ros2_control name="${name}" type="system">
       <hardware>
-        <plugin>gazebo_ros2_control/GazeboSystem</plugin>
+        <plugin>gz_ros2_control/GazeboSimSystem</plugin>
       </hardware>
       <joint name="joint_b">

File: aprs_description/urdf/motoman/motoman_sia20_macro.xacro (robot description, xacro)
@@ -8,4 +8,5 @@
 			<inertial>
 				<mass value="1.0"/>
+				<!--xacro:inertia_origin_base_link/-->
 				<inertia ixx="0.0226667" ixy="0.0" ixz="0.0" iyy="0.0226667" iyz="0.0" izz="0.0226667" />
 			</inertial>

File: aprs_description/urdf/ur/aprs_ur.ros2_control.xacro (robot description, xacro)
@@ -6,5 +6,5 @@
     <ros2_control name="${name}" type="system">
       <hardware>
-        <plugin>gazebo_ros2_control/GazeboSystem</plugin>
+        <plugin>gz_ros2_control/GazeboSimSystem</plugin>
       </hardware>
       <joint name="shoulder_pan_joint">

Commit message: Changes for Jazzy

File: aprs_description/urdf/aprs_lab_robots.urdf.xacro (robot description, xacro)
@@ -21,5 +21,5 @@
   </joint>
   <joint name = "motoman_world_to_base" type = "fixed">
-    <origin rpy = "0 0 3.14159" xyz = "0.4953 -0.08255 0.84455"/>
+    <origin rpy = "0 0 3.14159" xyz = "0.4953 -0.08255 0.9"/>
     <parent link = "world"/>
     <child link = "aprs_motoman_base_link"/>

File: aprs_description/urdf/aprs_motoman.urdf.xacro (robot description, xacro)
@@ -4,5 +4,5 @@
   <link name="aprs_motoman_base_link"/>
   <joint name = "motoman_world_to_base" type = "fixed">
-    <origin rpy = "0 0 3.14159" xyz = "0.4953 -0.08255 0.84455"/>
+    <origin rpy = "0 0 3.14159" xyz = "0.4953 -0.08255 0.9"/>
     <parent link = "world"/>
     <child link = "aprs_motoman_base_link"/>

File: aprs_description/urdf/fanuc/aprs_fanuc.ros2_control.xacro (robot description, xacro)
@@ -10,6 +10,6 @@
       <joint name="joint_1">
         <command_interface name="position">
-          <param name="min">{-2*pi}</param>
-          <param name="max">{2*pi}</param>
+          <param name="min">${-2*pi}</param>
+          <param name="max">${2*pi}</param>
         </command_interface>
         <state_interface name="position">
@@ -21,6 +21,6 @@
       <joint name="joint_2">
         <command_interface name="position">
-         <param name="min">{-2*pi}</param>
-          <param name="max">{2*pi}</param>
+         <param name="min">${-2*pi}</param>
+          <param name="max">${2*pi}</param>
         </command_interface>
         <state_interface name="position">
@@ -32,6 +32,6 @@
       <joint name="joint_3">
         <command_interface name="position">
-          <param name="min">{-pi}</param>
-          <param name="max">{pi}</param>
+          <param name="min">${-pi}</param>
+          <param name="max">${pi}</param>
         </command_interface>
         <state_interface name="position">
@@ -43,6 +43,6 @@
       <joint name="joint_4">
         <command_interface name="position">
-          <param name="min">{-2*pi}</param>
-          <param name="max">{2*pi}</param>
+          <param name="min">${-2*pi}</param>
+          <param name="max">${2*pi}</param>
         </command_interface>
         <state_interface name="position">
@@ -54,6 +54,6 @@
       <joint name="joint_5">
         <command_interface name="position">
-          <param name="min">{-2*pi}</param>
-          <param name="max">{2*pi}</param>
+          <param name="min">${-2*pi}</param>
+          <param name="max">${2*pi}</param>
         </command_interface>
         <state_interface name="position">
@@ -65,6 +65,6 @@
       <joint name="joint_6">
         <command_interface name="position">
-          <param name="min">{-2*pi}</param>
-          <param name="max">{2*pi}</param>
+          <param name="min">${-2*pi}</param>
+          <param name="max">${2*pi}</param>
         </command_interface>
         <state_interface name="position">

File: aprs_description/urdf/fanuc/aprs_fanuc_macro.xacro (robot description, xacro)
@@ -21,9 +21,9 @@
     </xacro:aprs_fanuc_ros2_control>
     <!-- Run gripper macro -->
-    <xacro:vacuum_gripper
+    <!-- <xacro:vacuum_gripper
       parent="fanuc_gripper_link"
       prefix="fanuc"
       >
-    </xacro:vacuum_gripper>
+    </xacro:vacuum_gripper> -->
   </xacro:macro>
 </robot>

File: aprs_description/urdf/motoman/aprs_motoman.ros2_control.xacro (robot description, xacro)
@@ -10,6 +10,6 @@
       <joint name="joint_b">
           <command_interface name="position">
-          <param name="min">{-2*pi}</param>
-          <param name="max">{2*pi}</param>
+          <param name="min">${-2*pi}</param>
+          <param name="max">${2*pi}</param>
           </command_interface>
           <state_interface name="position">
@@ -21,6 +21,6 @@
       <joint name="joint_e">
           <command_interface name="position">
-          <param name="min">{-2*pi}</param>
-          <param name="max">{2*pi}</param>
+          <param name="min">${-2*pi}</param>
+          <param name="max">${2*pi}</param>
           </command_interface>
           <state_interface name="position">
@@ -32,6 +32,6 @@
       <joint name="joint_l">
           <command_interface name="position">
-          <param name="min">{-pi}</param>
-          <param name="max">{pi}</param>
+          <param name="min">${-pi}</param>
+          <param name="max">${pi}</param>
           </command_interface>
           <state_interface name="position">
@@ -43,6 +43,6 @@
       <joint name="joint_r">
           <command_interface name="position">
-          <param name="min">{-2*pi}</param>
-          <param name="max">{2*pi}</param>
+          <param name="min">${-2*pi}</param>
+          <param name="max">${2*pi}</param>
           </command_interface>
           <state_interface name="position">
@@ -54,6 +54,6 @@
       <joint name="joint_s">
           <command_interface name="position">
-          <param name="min">{-2*pi}</param>
-          <param name="max">{2*pi}</param>
+          <param name="min">${-2*pi}</param>
+          <param name="max">${2*pi}</param>
           </command_interface>
           <state_interface name="position">
@@ -65,6 +65,6 @@
       <joint name="joint_t">
           <command_interface name="position">
-          <param name="min">{-2*pi}</param>
-          <param name="max">{2*pi}</param>
+          <param name="min">${-2*pi}</param>
+          <param name="max">${2*pi}</param>
           </command_interface>
           <state_interface name="position">
@@ -76,6 +76,6 @@
       <joint name="joint_u">
           <command_interface name="position">
-          <param name="min">{-2*pi}</param>
-          <param name="max">{2*pi}</param>
+          <param name="min">${-2*pi}</param>
+          <param name="max">${2*pi}</param>
           </command_interface>
           <state_interface name="position">

File: aprs_description/urdf/motoman/aprs_motoman_macro.xacro (robot description, xacro)
@@ -21,9 +21,9 @@
     </xacro:aprs_motoman_ros2_control>
     <!-- Run gripper macro -->
-    <xacro:vacuum_gripper
+    <!-- <xacro:vacuum_gripper
       parent="motoman_gripper_link"
       prefix="motoman"
       >
-    </xacro:vacuum_gripper>
+    </xacro:vacuum_gripper> -->
   </xacro:macro>
 </robot>

File: aprs_description/urdf/ur/aprs_ur.ros2_control.xacro (robot description, xacro)
@@ -10,6 +10,6 @@
       <joint name="shoulder_pan_joint">
         <command_interface name="position">
-          <param name="min">{-2*pi}</param>
-          <param name="max">{2*pi}</param>
+          <param name="min">${-2*pi}</param>
+          <param name="max">${2*pi}</param>
         </command_interface>
         <state_interface name="position">
@@ -22,6 +22,6 @@
       <joint name="shoulder_lift_joint">
         <command_interface name="position">
-          <param name="min">{-2*pi}</param>
-          <param name="max">{2*pi}</param>
+          <param name="min">${-2*pi}</param>
+          <param name="max">${2*pi}</param>
         </command_interface>
         <state_interface name="position">
@@ -34,6 +34,6 @@
       <joint name="elbow_joint">
         <command_interface name="position">
-          <param name="min">{-pi}</param>
-          <param name="max">{pi}</param>
+          <param name="min">${-pi}</param>
+          <param name="max">${pi}</param>
         </command_interface>
         <state_interface name="position">
@@ -46,6 +46,6 @@
       <joint name="wrist_1_joint">
         <command_interface name="position">
-          <param name="min">{-2*pi}</param>
-          <param name="max">{2*pi}</param>
+          <param name="min">${-2*pi}</param>
+          <param name="max">${2*pi}</param>
         </command_interface>
         <state_interface name="position">
@@ -58,6 +58,6 @@
       <joint name="wrist_2_joint">
         <command_interface name="position">
-          <param name="min">{-2*pi}</param>
-          <param name="max">{2*pi}</param>
+          <param name="min">${-2*pi}</param>
+          <param name="max">${2*pi}</param>
         </command_interface>
         <state_interface name="position">
@@ -70,6 +70,6 @@
       <joint name="wrist_3_joint">
         <command_interface name="position">
-          <param name="min">{-2*pi}</param>
-          <param name="max">{2*pi}</param>
+          <param name="min">${-2*pi}</param>
+          <param name="max">${2*pi}</param>
         </command_interface>
         <state_interface name="position">

File: aprs_description/urdf/ur/aprs_ur_macro.xacro (robot description, xacro)
@@ -28,9 +28,9 @@
     </xacro:aprs_ur_ros2_control>
     <!-- Run gripper macro -->
-    <xacro:vacuum_gripper
+    <!-- <xacro:vacuum_gripper
       parent="tool0"
       prefix="ur"
       >
-    </xacro:vacuum_gripper>
+    </xacro:vacuum_gripper> -->
   </xacro:macro>
 </robot>
