Commit message: Controllers working with combined and seperate descriptions

File: aprs_description/urdf/aprs_fanuc.urdf.xacro (robot description, xacro)
@@ -9,5 +9,5 @@
   </joint>
   <xacro:include filename="$(find aprs_description)/urdf/fanuc/aprs_fanuc_macro.xacro"/>
-  <xacro:arg name="fanuc_controller" default="$(find aprs_description)/config/individual_controllers/fanuc_controller.yaml" />
+  <xacro:arg name="fanuc_controller" default="$(find aprs_description)/config/robot_controllers.yaml" />
   <!-- <xacro:arg name="controllers" default="$(find aprs_description)/config/ns_robot_controllers.yaml" /> -->
   <xacro:aprs_fanuc
@@ -16,10 +16,9 @@
   <gazebo>
     <plugin filename="libgz_ros2_control-system.so" name="gz_ros2_control::GazeboSimROS2ControlPlugin">
-      <!-- <ros>
+      <ros>
         <namespace>fanuc</namespace>
-      </ros> -->
+      </ros>
+      <!-- <robot_param_node>fanuc_state_publisher</robot_param_node> -->
       <parameters>$(arg fanuc_controller)</parameters>
-      <load_params_directly>true</load_params_directly>
-      <controller name="joint_trajectory_controller" params_file="$(find aprs_description)/config/individual_controllers/fanuc_controller.yaml"/>
     </plugin>
   </gazebo>

File: aprs_description/urdf/aprs_franka.urdf.xacro (robot description, xacro)
@@ -9,15 +9,13 @@
   <xacro:include filename="$(find aprs_description)/urdf/franka/aprs_franka_macro.xacro"/>
     <!-- ROS2 Control Plugin -->
-  <xacro:arg name="franka_controller" default="$(find aprs_description)/config/individual_controllers/franka_controller.yaml" />
+  <xacro:arg name="franka_controller" default="$(find aprs_description)/config/robot_controllers.yaml" />
   <!-- <xacro:arg name="controllers" default="$(find aprs_description)/config/ns_robot_controllers.yaml" /> -->
   <xacro:aprs_franka></xacro:aprs_franka>
   <gazebo>
     <plugin filename="libgz_ros2_control-system.so" name="gz_ros2_control::GazeboSimROS2ControlPlugin">
-      <!-- <ros>
+      <ros>
         <namespace>franka</namespace>
-      </ros> -->
+      </ros>
       <parameters>$(arg franka_controller)</parameters>
-      <load_params_directly>true</load_params_directly>
-      <controller name="joint_trajectory_controller" params_file="$(find aprs_description)/config/individual_controllers/franka_controller.yaml"/>
     </plugin>
   </gazebo>

File: aprs_description/urdf/aprs_lab_robots.urdf.xacro (robot description, xacro)
@@ -47,8 +47,4 @@
       <parameters>$(arg controllers)</parameters>
       <load_params_directly>true</load_params_directly>
-      <controller name="ur_joint_trajectory_controller" params_file="$(find aprs_description)/config/robot_controllers.yaml"/>
-      <controller name="franka_joint_trajectory_controller" params_file="$(find aprs_description)/config/robot_controllers.yaml"/>
-      <controller name="fanuc_joint_trajectory_controller" params_file="$(find aprs_description)/config/robot_controllers.yaml"/>
-      <controller name="motoman_joint_trajectory_controller" params_file="$(find aprs_description)/config/robot_controllers.yaml"/>
     </plugin>
   </gazebo>

File: aprs_description/urdf/aprs_motoman.urdf.xacro (robot description, xacro)
@@ -10,6 +10,6 @@
   <xacro:include filename="$(find aprs_description)/urdf/motoman/aprs_motoman_macro.xacro"/>
     <!-- ROS2 Control Plugin -->
-  <xacro:arg name="motoman_controller" default="$(find aprs_description)/config/individual_controllers/motoman_controller.yaml" />
-  <!-- <xacro:arg name="controllers" default="$(find aprs_description)/config/ns_robot_controllers.yaml" /> -->
+  <!-- <xacro:arg name="motoman_controller" default="$(find aprs_description)/config/individual_controllers/motoman_controller.yaml" /> -->
+  <xacro:arg name="motoman_controller" default="$(find aprs_description)/config/robot_controllers.yaml" />
   <xacro:aprs_motoman
     parent="aprs_motoman_base_link">
@@ -17,10 +17,8 @@
   <gazebo>
     <plugin filename="libgz_ros2_control-system.so" name="gz_ros2_control::GazeboSimROS2ControlPlugin">
-      <!-- <ros>
+      <ros>
         <namespace>motoman</namespace>
-      </ros> -->
+      </ros>
       <parameters>$(arg motoman_controller)</parameters>
-      <load_params_directly>true</load_params_directly>
-      <controller name="joint_trajectory_controller" params_file="$(find aprs_description)/config/individual_controllers/motoman_controller.yaml"/>
     </plugin>
   </gazebo>

File: aprs_description/urdf/aprs_ur.urdf.xacro (robot description, xacro)
@@ -10,5 +10,5 @@
   <xacro:include filename="$(find aprs_description)/urdf/ur/aprs_ur_macro.xacro"/>
     <!-- ROS2 Control Plugin -->
-  <xacro:arg name="ur_controller" default="$(find aprs_description)/config/individual_controllers/ur_controller.yaml" />
+  <xacro:arg name="ur_controller" default="$(find aprs_description)/config/robot_controllers.yaml" />
   <!-- <xacro:arg name="controllers" default="$(find aprs_description)/config/ns_robot_controllers.yaml" /> -->
   <xacro:aprs_ur
@@ -17,10 +17,8 @@
   <gazebo>
     <plugin filename="libgz_ros2_control-system.so" name="gz_ros2_control::GazeboSimROS2ControlPlugin">
-      <!-- <ros>
+      <ros>
         <namespace>ur</namespace>
-      </ros> -->
+      </ros>
       <parameters>$(arg ur_controller)</parameters>
-      <load_params_directly>true</load_params_directly>
-      <controller name="joint_trajectory_controller" params_file="$(find aprs_description)/config/individual_controllers/ur_controller.yaml"/>
     </plugin>
   </gazebo>

File: aprs_description/urdf/franka/aprs_franka.ros2_control.xacro (robot description, xacro)
@@ -85,4 +85,14 @@
         <state_interface name="effort"/>
       </joint>
+      <joint name="fr3_finger_joint1">
+        <state_interface name="position"></state_interface>
+        <state_interface name="velocity"/>
+        <state_interface name="effort"/>
+      </joint>
+      <joint name="fr3_finger_joint2">
+        <state_interface name="position"></state_interface>
+        <state_interface name="velocity"/>
+        <state_interface name="effort"/>
+      </joint>
     </ros2_control>
   </xacro:macro>

Commit message: Robots with vacuum gripper can spawn in with cameras

File: aprs_description/urdf/aprs_fanuc.urdf.xacro (robot description, xacro)
@@ -11,6 +11,13 @@
   <xacro:arg name="fanuc_controller" default="$(find aprs_description)/config/robot_controllers.yaml" />
   <!-- <xacro:arg name="controllers" default="$(find aprs_description)/config/ns_robot_controllers.yaml" /> -->
+  <xacro:arg name="camera_active_arg" default="false"/>
+  <xacro:property name="camera_active" value="$(arg camera_active_arg)" />
+  <xacro:arg name="camera_type_arg" default="rgb"/>
+  <xacro:property name="camera_type" value="$(arg camera_type_arg)" />
   <xacro:aprs_fanuc
-    parent="aprs_fanuc_base_link">
+    parent="aprs_fanuc_base_link"
+    camera_active="${camera_active}"
+    camera_type="${camera_type}"
+    >
   </xacro:aprs_fanuc>
   <gazebo>

File: aprs_description/urdf/aprs_lab_robots.urdf.xacro (robot description, xacro)
@@ -31,13 +31,34 @@
     <!-- ROS2 Control Plugin -->
   <xacro:arg name="controllers" default="$(find aprs_description)/config/robot_controllers.yaml" />
+  <xacro:arg name="ur_camera_active_arg" default="false"/>
+  <xacro:property name="ur_camera_active" value="$(arg ur_camera_active_arg)" />
+  <xacro:arg name="ur_camera_type_arg" default="rgb"/>
+  <xacro:property name="ur_camera_type" value="$(arg ur_camera_type_arg)" />
   <xacro:aprs_ur
-    parent="aprs_ur_base_link">
+    parent="aprs_ur_base_link"
+    camera_active="${ur_camera_active}"
+    camera_type="${ur_camera_type}"
+    >
   </xacro:aprs_ur>
+  <xacro:arg name="fanuc_camera_active_arg" default="false"/>
+  <xacro:property name="fanuc_camera_active" value="$(arg fanuc_camera_active_arg)" />
+  <xacro:arg name="fanuc_camera_type_arg" default="rgb"/>
+  <xacro:property name="fanuc_camera_type" value="$(arg fanuc_camera_type_arg)" />
   <xacro:aprs_fanuc
-    parent="aprs_fanuc_base_link">
+    parent="aprs_fanuc_base_link"
+    camera_active="${fanuc_camera_active}"
+    camera_type="${fanuc_camera_type}"
+    >
   </xacro:aprs_fanuc>
   <xacro:aprs_franka></xacro:aprs_franka>
+  <xacro:arg name="motoman_camera_active_arg" default="false"/>
+  <xacro:property name="motoman_camera_active" value="$(arg motoman_camera_active_arg)" />
+  <xacro:arg name="motoman_camera_type_arg" default="rgb"/>
+  <xacro:property name="motoman_camera_type" value="$(arg motoman_camera_type_arg)" />
   <xacro:aprs_motoman
-    parent="aprs_motoman_base_link">
+    parent="aprs_motoman_base_link"
+    camera_active="${motoman_camera_active}"
+    camera_type="${motoman_camera_type}"
+    >
   </xacro:aprs_motoman>
   <gazebo>

File: aprs_description/urdf/aprs_motoman.urdf.xacro (robot description, xacro)
@@ -12,6 +12,13 @@
   <!-- <xacro:arg name="motoman_controller" default="$(find aprs_description)/config/individual_controllers/motoman_controller.yaml" /> -->
   <xacro:arg name="motoman_controller" default="$(find aprs_description)/config/robot_controllers.yaml" />
+  <xacro:arg name="camera_active_arg" default="false"/>
+  <xacro:property name="camera_active" value="$(arg camera_active_arg)" />
+  <xacro:arg name="camera_type_arg" default="rgb"/>
+  <xacro:property name="camera_type" value="$(arg camera_type_arg)" />
   <xacro:aprs_motoman
-    parent="aprs_motoman_base_link">
+    parent="aprs_motoman_base_link"
+    camera_active="${camera_active}"
+    camera_type="${camera_type}"
+    >
   </xacro:aprs_motoman>
   <gazebo>

File: aprs_description/urdf/aprs_ur.urdf.xacro (robot description, xacro)
@@ -12,6 +12,13 @@
   <xacro:arg name="ur_controller" default="$(find aprs_description)/config/robot_controllers.yaml" />
   <!-- <xacro:arg name="controllers" default="$(find aprs_description)/config/ns_robot_controllers.yaml" /> -->
+  <xacro:arg name="camera_active_arg" default="false"/>
+  <xacro:property name="camera_active" value="$(arg camera_active_arg)" />
+  <xacro:arg name="camera_type_arg" default="rgb"/>
+  <xacro:property name="camera_type" value="$(arg camera_type_arg)" />
   <xacro:aprs_ur
-    parent="aprs_ur_base_link">
+    parent="aprs_ur_base_link"
+    camera_active="${camera_active}"
+    camera_type="${camera_type}"
+    >
   </xacro:aprs_ur>
   <gazebo>

File: aprs_description/urdf/fanuc/aprs_fanuc_macro.xacro (robot description, xacro)
@@ -3,4 +3,6 @@
   <xacro:macro name="aprs_fanuc" params="
     parent
+    camera_active
+    camera_type
 ">
     <!-- Inclue fanuc robot macro -->
@@ -21,9 +23,11 @@
     </xacro:aprs_fanuc_ros2_control>
     <!-- Run gripper macro -->
-    <!-- <xacro:vacuum_gripper
+    <xacro:vacuum_gripper
       parent="fanuc_gripper_link"
       prefix="fanuc"
+      use_camera="${camera_active}"
+      camera_type="${camera_type}"
       >
-    </xacro:vacuum_gripper> -->
+    </xacro:vacuum_gripper>
   </xacro:macro>
 </robot>

File: aprs_description/urdf/motoman/aprs_motoman_macro.xacro (robot description, xacro)
@@ -3,4 +3,6 @@
   <xacro:macro name="aprs_motoman" params="
     parent
+    camera_active
+    camera_type
 ">
     <!-- Inclue motoman robot macro -->
@@ -21,9 +23,11 @@
     </xacro:aprs_motoman_ros2_control>
     <!-- Run gripper macro -->
-    <!-- <xacro:vacuum_gripper
+    <xacro:vacuum_gripper
       parent="motoman_gripper_link"
       prefix="motoman"
+      use_camera="${camera_active}"
+      camera_type="${camera_type}"
       >
-    </xacro:vacuum_gripper> -->
+    </xacro:vacuum_gripper>
   </xacro:macro>
 </robot>

File: aprs_description/urdf/ur/aprs_ur_macro.xacro (robot description, xacro)
@@ -3,4 +3,6 @@
   <xacro:macro name="aprs_ur" params="
     parent
+    camera_active
+    camera_type
 ">
     <!-- Inclue ur robot macro -->
@@ -28,9 +30,11 @@
     </xacro:aprs_ur_ros2_control>
     <!-- Run gripper macro -->
-    <!-- <xacro:vacuum_gripper
+    <xacro:vacuum_gripper
       parent="tool0"
       prefix="ur"
+      use_camera="${camera_active}"
+      camera_type="${camera_type}"
       >
-    </xacro:vacuum_gripper> -->
+    </xacro:vacuum_gripper>
   </xacro:macro>
 </robot>

File: aprs_description/urdf/vacuum_gripper/vacuum_grippper_macro.xacro (robot description, xacro)
@@ -4,4 +4,6 @@
     parent
     prefix
+    use_camera
+    camera_type
     ">
     <!-- Gripper Link -->
@@ -12,5 +14,4 @@
           <mesh filename="file://$(find aprs_description)/meshes/vacuum_gripper/vacuum_gripper.stl" scale="1 1 1"/>
         </geometry>
-        <material name="Grey"/>
       </visual>
       <collision name="${prefix}_gripper_collision">
@@ -45,5 +46,5 @@
     </gazebo>
     <!-- ROS2 Control for the gripper joint -->
-    <ros2_control name="${prefix}_gripper_control" type="system">
+    <!-- <ros2_control name="${prefix}_gripper_control" type="system">
       <hardware>
         <plugin>gazebo_ros2_control/GazeboSystem</plugin>
@@ -54,5 +55,5 @@
         </state_interface>
       </joint>
-    </ros2_control>
+    </ros2_control> -->
     <!-- Vacuum gripper plugin
     <gazebo>
@@ -64,4 +65,127 @@
       </plugin>
     </gazebo> -->
+    <!-- Camera -->
+    <xacro:if value="${use_camera}">
+      <!-- Mount Link -->
+      <link name ="${prefix}_robot_camera_mount_link">
+        <visual>
+          <origin xyz="0 0 0" rpy="0 0 0"/>
+          <geometry>
+            <mesh filename="file://$(find aprs_description)/meshes/vacuum_gripper/camera_mount.stl" scale="1 1 1"/>
+          </geometry>
+        </visual>
+      </link>
+      <!-- Camera Link -->
+      <link name ="${prefix}_robot_camera_link">
+        <visual>
+          <origin xyz="0 0 0" rpy="1.57 0 1.57"/>
+          <geometry>
+            <mesh filename="file://$(find aprs_description)/meshes/vacuum_gripper/camera.stl" scale="1 1 1"/>
+          </geometry>
+        </visual>
+      </link>
+      <link name ="${prefix}_robot_camera_optical_link">
+      </link>
+      <!-- Add camera mount joint -->
+      <joint name="${prefix}_robot_camera_mount_joint" type="fixed">
+        <axis xyz="0 1 0" />
+        <origin xyz="0 0 -0.012" rpy="0 0 0"/>
+        <parent link="${prefix}_gripper"/>
+        <child link="${prefix}_robot_camera_mount_link"/>
+      </joint>
+      <!-- Add camera joint -->
+      <joint name="${prefix}_robot_camera_joint" type="fixed">
+        <axis xyz="0 1 0" />
+        <origin xyz="0 -.07 -.006" rpy="0 -1.57 1.57"/>
+        <parent link="${prefix}_robot_camera_mount_link"/>
+        <child link="${prefix}_robot_camera_link"/>
+      </joint>
+      <!-- Add optical joint -->
+      <joint name="${prefix}_robot_camera_optical_joint" type="fixed">
+        <axis xyz="0 1 0" />
+        <origin xyz="0 0 0" rpy="-1.57 0 -1.57"/>
+        <parent link="${prefix}_robot_camera_link"/>
+        <child link="${prefix}_robot_camera_optical_link"/>
+      </joint>
+      <!-- Add color to links -->
+      <gazebo reference="${prefix}_robot_camera_mount_link">
+        <material>Gazebo/Black</material>
+      </gazebo>
+      <gazebo reference="${prefix}_robot_camera_link">
+        <material>Gazebo/White</material>
+      </gazebo>
+      <!-- Add gazebo sensors -->
+      <xacro:property name="type" value="${camera_type}"/>
+      <gazebo reference="${prefix}_robot_camera_link">
+        <!-- Add rgb camera -->
+        <xacro:if value="${type == 'rgb'}">
+          <sensor type="camera" name="rgb_camera">
+            <topic>${prefix}_robot_rgb_camera_gz_topic</topic>
+            <always_on>true</always_on>
+            <visualize>false</visualize>
+            <update_rate>15</update_rate>
+            <camera name="${prefix}_robot_camera">
+              <horizontal_fov>1.5</horizontal_fov>
+              <image>
+                <width>640</width>
+                <height>480</height>
+                <format>R8G8B8</format>
+              </image>
+              <clip>
+                <near>0.1</near>
+                <far>10</far>
+              </clip>
+            </camera>
+            <plugin name="ariac_sensors::AriacCameraPlugin" filename="libAriacCameraPlugin.so">
+              <ros>
+                <namespace></namespace>
+              </ros>
+              <camera_type>rgb</camera_type>
+              <gz_topic>${prefix}_robot_rgb_camera_gz_topic</gz_topic>
+              <camera_name>${prefix}_robot_rgb_camera</camera_name>
+              <rgb_img_ros_topic>/ariac/sensors/${prefix}_robot_rgb_camera/rgb_image</rgb_img_ros_topic>
+              <cam_info_ros_topic>/ariac/sensors/${prefix}_robot_rgb_camera/camera_info</cam_info_ros_topic>
+              <cam_info_gz_topic>${prefix}_robot_rgb_camera_gz_topic_info</cam_info_gz_topic>
+            </plugin>
+          </sensor>
+        </xacro:if>
+        <xacro:if value="${type == 'rgbd'}">
+          <sensor type="depth" name="rgbd_camera">
+            <topic>${prefix}_robot_rgbd_camera_gz_topic</topic>
+            <always_on>true</always_on>
+            <visualize>false</visualize>
+            <update_rate>15</update_rate>
+            <camera name="${prefix}_robot_camera">
+              <horizontal_fov>1.5</horizontal_fov>
+              <image>
+                <width>640</width>
+                <height>480</height>
+                <format>R8G8B8</format>
+              </image>
+              <clip>
+                <near>0.1</near>
+                <far>10</far>
+              </clip>
+              <noise>
+                <type>gaussian</type>
+                <mean>0.0</mean>
+                <stddev>0.001</stddev>
+              </noise>
+            </camera>
+            <plugin name="ariac_sensors::AriacCameraPlugin" filename="libAriacCameraPlugin.so">
+              <ros>
+                <namespace></namespace>
+              </ros>
+              <camera_type>rgbd</camera_type>
+              <camera_name>${prefix}_robot_rgbd_camera</camera_name>
+              <gz_topic>${prefix}_robot_rgbd_camera_gz_topic</gz_topic>
+              <rgb_img_ros_topic>/ariac/sensors/${prefix}_robot_rgbd_camera/rgb_image</rgb_img_ros_topic>
+              <depth_img_ros_topic>/ariac/sensors/${prefix}_robot_rgbd_camera/depth_image</depth_img_ros_topic>
+              <cam_info_ros_topic>/ariac/sensors/${prefix}_robot_rgbd_camera/camera_info</cam_info_ros_topic>
+            </plugin>
+          </sensor>
+        </xacro:if>
+      </gazebo>
+    </xacro:if>
   </xacro:macro>
 </robot>
