Commit message: Changes

File: aprs_description/urdf/aprs_fanuc.urdf.xacro (robot description, xacro)
@@ -10,5 +10,4 @@
   <xacro:include filename="$(find aprs_description)/urdf/fanuc/aprs_fanuc_macro.xacro"/>
   <xacro:arg name="fanuc_controller" default="$(find aprs_description)/config/robot_controllers.yaml" />
-  <!-- <xacro:arg name="controllers" default="$(find aprs_description)/config/ns_robot_controllers.yaml" /> -->
   <xacro:arg name="camera_active_arg" default="false"/>
   <xacro:property name="camera_active" value="$(arg camera_active_arg)" />
@@ -27,7 +26,5 @@
       </ros>
       <parameters>$(arg fanuc_controller)</parameters>
-      <!-- <controller_manager_name>fanuc_controller_manager</controller_manager_name> -->
       <robot_param>robot_description</robot_param>
-      <!-- <robot_param_node>/fanuc/robot_state_publisher</robot_param_node> -->
     </plugin>
   </gazebo>

File: aprs_description/urdf/aprs_franka.urdf.xacro (robot description, xacro)
@@ -8,7 +8,5 @@
   </joint>
   <xacro:include filename="$(find aprs_description)/urdf/franka/aprs_franka_macro.xacro"/>
-    <!-- ROS2 Control Plugin -->
   <xacro:arg name="franka_controller" default="$(find aprs_description)/config/robot_controllers.yaml" />
-  <!-- <xacro:arg name="controllers" default="$(find aprs_description)/config/ns_robot_controllers.yaml" /> -->
   <xacro:aprs_franka></xacro:aprs_franka>
   <gazebo>
@@ -18,7 +16,5 @@
       </ros>
       <parameters>$(arg franka_controller)</parameters>
-      <!-- <controller_manager_name>franka_controller_manager</controller_manager_name> -->
       <robot_param>robot_description</robot_param>
-      <!-- <robot_param_node>/franka/robot_state_publisher</robot_param_node> -->
     </plugin>
   </gazebo>

File: aprs_description/urdf/aprs_lab_robots.urdf.xacro (robot description, xacro)
@@ -29,5 +29,4 @@
   <xacro:include filename="$(find aprs_description)/urdf/franka/aprs_franka_macro.xacro"/>
   <xacro:include filename="$(find aprs_description)/urdf/motoman/aprs_motoman_macro.xacro"/>
-    <!-- ROS2 Control Plugin -->
   <xacro:arg name="controllers" default="$(find aprs_description)/config/robot_controllers.yaml" />
   <xacro:arg name="ur_camera_active_arg" default="false"/>

File: aprs_description/urdf/aprs_motoman.urdf.xacro (robot description, xacro)
@@ -9,6 +9,4 @@
   </joint>
   <xacro:include filename="$(find aprs_description)/urdf/motoman/aprs_motoman_macro.xacro"/>
-    <!-- ROS2 Control Plugin -->
-  <!-- <xacro:arg name="motoman_controller" default="$(find aprs_description)/config/individual_controllers/motoman_controller.yaml" /> -->
   <xacro:arg name="motoman_controller" default="$(find aprs_description)/config/robot_controllers.yaml" />
   <xacro:arg name="camera_active_arg" default="false"/>
@@ -28,7 +26,5 @@
       </ros>
       <parameters>$(arg motoman_controller)</parameters>
-      <!-- <controller_manager_name>motoman_controller_manager</controller_manager_name> -->
       <robot_param>robot_description</robot_param>
-      <!-- <robot_param_node>/motoman/robot_state_publisher</robot_param_node> -->
     </plugin>
   </gazebo>

File: aprs_description/urdf/aprs_ur.urdf.xacro (robot description, xacro)
@@ -9,7 +9,5 @@
   </joint>
   <xacro:include filename="$(find aprs_description)/urdf/ur/aprs_ur_macro.xacro"/>
-    <!-- ROS2 Control Plugin -->
   <xacro:arg name="ur_controller" default="$(find aprs_description)/config/robot_controllers.yaml" />
-  <!-- <xacro:arg name="controllers" default="$(find aprs_description)/config/ns_robot_controllers.yaml" /> -->
   <xacro:arg name="camera_active_arg" default="false"/>
   <xacro:property name="camera_active" value="$(arg camera_active_arg)" />
@@ -28,7 +26,5 @@
       </ros>
       <parameters>$(arg ur_controller)</parameters>
-      <!-- <controller_manager_name>ur_controller_manager</controller_manager_name> -->
       <robot_param>robot_description</robot_param>
-      <!-- <robot_param_node>/ur/robot_state_publisher</robot_param_node> -->
     </plugin>
   </gazebo>

File: aprs_description/urdf/vacuum_gripper/vacuum_gripper_macro.xacro (robot description, xacro)
@@ -50,24 +50,4 @@
       </sensor>
     </gazebo>
-    <!-- ROS2 Control for the gripper joint -->
-    <!-- <ros2_control name="${prefix}_gripper_control" type="system">
-      <hardware>
-        <plugin>gazebo_ros2_control/GazeboSystem</plugin>
-      </hardware>
-      <joint name="${prefix}_gripper_joint">
-        <state_interface name="position">
-          <param name="initial_value">0</param>
-        </state_interface>
-      </joint>
-    </ros2_control> -->
-    <!-- Vacuum gripper plugin
-    <gazebo>
-      <plugin filename="libVacuumGripperPlugin.so" name="${prefix}_vacuum_gripper_plugin">
-        <ros>
-        </ros>
-        <gripper_link>${prefix}_gripper</gripper_link>
-        <robot_name>${prefix}_robot</robot_name>
-      </plugin>
-    </gazebo> -->
     <!-- Camera -->
     <xacro:if value="${use_camera}">

Commit message: Conveyor is the problem

File: aprs_description/urdf/aprs_fanuc.urdf.xacro (robot description, xacro)
@@ -26,4 +26,5 @@
       </ros>
       <parameters>$(arg fanuc_controller)</parameters>
+      <load_params_directly>true</load_params_directly>
       <robot_param>robot_description</robot_param>
     </plugin>

File: aprs_description/urdf/aprs_motoman.urdf.xacro (robot description, xacro)
@@ -2,4 +2,7 @@
 <robot xmlns:xacro="http://www.ros.org/wiki/xacro" name="aprs_lab_robots">
   <link name="world"/>
+  <gazebo
+      reference="world">
+  </gazebo>
   <link name="aprs_motoman_base_link"/>
   <joint name = "motoman_world_to_base" type = "fixed">
@@ -26,4 +29,5 @@
       </ros>
       <parameters>$(arg motoman_controller)</parameters>
+      <load_params_directly>true</load_params_directly>
       <robot_param>robot_description</robot_param>
     </plugin>

File: aprs_description/urdf/aprs_ur.urdf.xacro (robot description, xacro)
@@ -9,23 +9,7 @@
   </joint>
   <xacro:include filename="$(find aprs_description)/urdf/ur/aprs_ur_macro.xacro"/>
-  <xacro:arg name="ur_controller" default="$(find aprs_description)/config/robot_controllers.yaml" />
-  <xacro:arg name="camera_active_arg" default="false"/>
-  <xacro:property name="camera_active" value="$(arg camera_active_arg)" />
-  <xacro:arg name="camera_type_arg" default="rgb"/>
-  <xacro:property name="camera_type" value="$(arg camera_type_arg)" />
   <xacro:aprs_ur
     parent="aprs_ur_base_link"
-    camera_active="${camera_active}"
-    camera_type="${camera_type}"
     >
   </xacro:aprs_ur>
-  <gazebo>
-    <plugin filename="libgz_ros2_control-system.so" name="gz_ros2_control::GazeboSimROS2ControlPlugin">
-      <ros>
-        <namespace>simulation/ur</namespace>
-      </ros>
-      <parameters>$(arg ur_controller)</parameters>
-      <robot_param>robot_description</robot_param>
-    </plugin>
-  </gazebo>
 </robot>

File: aprs_description/urdf/motoman/aprs_motoman.ros2_control.xacro (robot description, xacro)
@@ -10,9 +10,9 @@
       <joint name="joint_b">
           <command_interface name="position">
-          <param name="min">${-2*pi}</param>
-          <param name="max">${2*pi}</param>
+            <param name="min">${-2*pi}</param>
+            <param name="max">${2*pi}</param>
           </command_interface>
           <state_interface name="position">
-          <param name="initial_value">${initial_positions['joint_b']}</param>
+            <param name="initial_value">${initial_positions['joint_b']}</param>
           </state_interface>
           <state_interface name="velocity"/>

File: aprs_description/urdf/ur/aprs_ur_macro.xacro (robot description, xacro)
@@ -3,6 +3,4 @@
   <xacro:macro name="aprs_ur" params="
     parent
-    camera_active
-    camera_type
 ">
     <!-- Inclue ur robot macro -->
@@ -10,7 +8,6 @@
     <!-- Include ROS2 Control macro -->
     <xacro:include filename="$(find aprs_description)/urdf/ur/aprs_ur.ros2_control.xacro"/>
-    <!-- Inclue gripper macro -->
-    <xacro:include filename="$(find aprs_description)/urdf/vacuum_gripper/vacuum_gripper_macro.xacro"/>
     <xacro:property name="initial_positions_file" default="$(find aprs_description)/config/ur_initial_positions.yaml"/>
+    <gazebo reference="${parent}"/>
     <!-- Run ur macro -->
     <xacro:ur_robot
@@ -29,6 +26,14 @@
       initial_positions="${xacro.load_yaml(initial_positions_file)}">
     </xacro:aprs_ur_ros2_control>
+    <gazebo>
+      <plugin filename="libgz_ros2_control-system" name="gz_ros2_control::GazeboSimROS2ControlPlugin">
+        <ros>
+          <namespace>simulation/ur</namespace>
+        </ros>
+        <parameters>$(find aprs_description)/config/robot_controllers.yaml</parameters>
+      </plugin>
+    </gazebo>
     <!-- Run gripper macro -->
-    <xacro:vacuum_gripper
+    <!-- <xacro:vacuum_gripper
       parent="tool0"
       prefix="ur"
@@ -36,5 +41,5 @@
       camera_type="${camera_type}"
       >
-    </xacro:vacuum_gripper>
+    </xacro:vacuum_gripper> -->
   </xacro:macro>
 </robot>
