Commit message: Worked on vacuum gripper

File: aprs_description/urdf/vacuum_gripper/vacuum_grippper_macro.xacro (robot description, xacro)
@@ -26,4 +26,9 @@
         <inertia ixx="0.0000647" ixy="0.0" ixz="0.0" iyy="0.0000647" iyz="0.0" izz="0.0001276"/>
       </inertial>
+      <sensor name='${prefix}_sensor_contact' type='contact'>
+        <contact>
+          <collision>"${prefix}_gripper_collision"</collision>
+        </contact>
+      </sensor>
     </link>
     <!-- Gripper Joint -->
